File: DataIO/DataROM/DataIOROM/decode.kicad_sch (KiCad schematic)
At the start: 10 parts, among them J10 Conn_02x08_Counter_Clockwise, J11 BANK3, J6 BANK0, J7 BANK1, J8 BANK2, J9 Conn_02x08_Counter_Clockwise, U2 SST39SF040_TSOP

Commit message: Tidy up v2.2 files
Parts:
- renumbered U2 to U1, J9 to U14, J10 to U19
