File: DataIO/DataROM/DataIOROM/rom.kicad_sch (KiCad schematic)
At the start: 14 parts, among them J1 Conn_01x03, J2 Conn_01x03, J3 Conn_01x03, J4 Conn_01x03, J5 Conn_01x03, U18 Conn_02x08_Counter_Clockwise, U2 SST39SF040_TSOP, U20 Conn_02x14_Counter_Clockwise, U3 GAL16V8, U7 Conn_02x08_Counter_Clockwise

Commit message: Tidy up v2.2 files
Parts:
- renumbered C2 to C1, C1 to C2, J3 to J2, J2 to J3, U18 to U180, U7 to U70
